Commit message: Change the joint limits on the grippers in the urdf

File: public/assets/pf400_description/urdf/PF400.urdf (robot description, URDF)
Before this commit: robot PF400_Robot, 9 links, 8 joints
Joints:
- joint J5: limit lower=0.067454 upper=0.070 effort=1000.0 velocity=0.5 -> lower=0.00 upper=0.070 effort=1000.0 velocity=0.5
- joint J5_mirror: limit lower=0.067454 upper=0.070 effort=1000.0 velocity=0.5 -> lower=0.00 upper=0.070 effort=1000.0 velocity=0.5

Commit message: Update urdf limits

File: public/assets/pf400_description/urdf/PF400.urdf (robot description, URDF)
Before this commit: robot PF400_Robot, 9 links, 8 joints
Joints:
- joint J1: limit lower=0.002 upper=1.160 effort=1000.0 velocity=0.5 -> lower=0.000 upper=1.160 effort=1000.0 velocity=0.5
- joint J3: limit lower=0.175 upper=6.1 effort=1000.0 velocity=0.5 -> lower=0.0 upper=6.1 effort=1000.0 velocity=0.5

Commit message: Update gripper limits

File: public/assets/pf400_description/urdf/PF400.urdf (robot description, URDF)
Before this commit: robot PF400_Robot, 9 links, 8 joints
Joints:
- joint J5: limit lower=0.00 upper=0.070 effort=1000.0 velocity=0.5 -> lower=0.00 upper=0.14 effort=1000.0 velocity=0.5
- joint J5_mirror: limit lower=0.00 upper=0.070 effort=1000.0 velocity=0.5 -> lower=0.00 upper=0.14 effort=1000.0 velocity=0.5
